File: twpatron.kicad_pcb (KiCad board)
At the start: 2 copper layers, 35.6 x 24.1 mm, 7 parts, among them J1 Conn_01x04, J2 Conn_Coaxial, J6 Conn_01x04, U1 MM5800, U2 MM5800, U3 MM5800, U4 MM5800

Commit message: twpatron added to powerpoint
Routing:
- net Net-(U1-RF2): track 0.00 -> 2.68 mm
- net Net-(U1-RF1): track 0.00 -> 2.68 mm
- net Net-(U3-RF2): track 0.00 -> 2.17 mm
Changed lines of the file:
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@@
+	)
+	(segment
+		(start 139.165237 99.53854)
+		(end 140.720373 101.093676)
+		(width 0.2)
+		(layer "F.Cu")
+		(net 2)
+	)
+	(segment
+		(start 138.738635 99.41354)
+		(end 138.863635 99.53854)
+		(width 0.2)
+		(layer "F.Cu")
+		(net 2)
+	)
+	(segment
+		(start 138.863635 99.53854)
+		(end 139.165237 99.53854)
+		(width 0.2)
+		(layer "F.Cu")
+		(net 2)
 	)
 	(segment
@@
 	)
 	(segment
+		(start 134.23 99.897001)
+		(end 134.105 99.772001)
+		(width 0.2)
+		(layer "F.Cu")
+		(net 4)
+	)
+	(segment
+		(start 134.105 99.557649)
+		(end 132.843675 98.296324)
+		(width 0.2)
+		(layer "F.Cu")
+		(net 4)
+	)
+	(segment
+		(start 134.105 99.772001)
+		(end 134.105 99.557649)
+		(width 0.2)
+		(layer "F.Cu")
+		(net 4)
+	)
+	(segment
+		(start 136.101174 100.615001)
+		(end 135.12 100.615001)
+		(width 0.2)
+		(layer "F.Cu")
+		(net 5)
+	)
+	(segment
+		(start 137.302635 99.41354)
+		(end 136.101174 100.615001)
+		(width 0.2)
+		(layer "F.Cu")
+		(net 5)
+	)
+	(segment
