File: twpatron-2.kicad_pcb (KiCad board)
At the start: 4 copper layers, 38.1 x 21 mm, 7 parts, among them J1 Conn_01x04, J3 SMP-straight-19S141-40ML5, J6 Conn_01x04, U1 MM5800, U2 MM5800, U3 MM5800, U4 MM5800

Commit message: twpatron2 close to a full draft
Parts:
- added ?: , , F.Cu at (155.7, 74.3)
- added ?: , , F.Cu at (132.9, 86.3)
- added ?: , , F.Cu at (143.0, 74.3)
- added ?: , , F.Cu at (165.9, 86.3)
- added R1: R_US, Resistor_SMD:R_0201_0603Metric, F.Cu at (140.2, 81.8)
Connections:
- U4 pad C1: unconnected-(U4-RF2-PadC1) -> Net-(U4-RF2)
- U4 pad C3: unconnected-(U4-RF1-PadC3) -> GND
Routing:
- net Net-(J1-Pin_1): track 30.7 -> 33.3 mm
- net Net-(U4-RF2): track 0.00 -> 1.32 mm
- net GND: vias 0 -> 87
Other:
- board text added: "1"
- board text added: "1+CAL"
- board text added: "2"
- board text added: "2+3"
- board text added: "3"
- board text added: "CAL"
- board text added: "LOAD"
- board text added: "SHORT"
