File: twpatron-2.kicad_sch (KiCad schematic)
At the start: 7 parts, among them J1 Conn_01x04, J3 SMP-straight-19S141-40ML5, J6 Conn_01x04, U1 MM5800, U2 MM5800, U3 MM5800, U4 MM5800

Commit message: twpatron2 close to a full draft
Parts:
- removed J3: SMP-straight-19S141-40ML5, rosenberger-smp:rosenberger-19S141-40ML5, symbol SchlibLafe:root_1_SMP-straight-19S141-40ML5_SchlibLafe.SchLib
- added J2: smp-straight, symbol Connector:Conn_Coaxial
- added R1: R_US, Resistor_SMD:R_0201_0603Metric, symbol Device:R_US
Connections:
- net GND: now also U4.C3 (RF1), J2.2 (Ext), R1.1
- net at U4.C1 (RF2): now also R1.2
- net at U1.A3 (RFC): now also J2.1 (In)
